File: Schematics/MotorTotem_Rev1/MotorTotem_Rev1/stepper.kicad_sch (KiCad schematic)
At the start: 13 parts, among them J2 Conn_01x04, J3 Conn_01x04, J4 Conn_01x04, U5 TMC2209_SILENTSTEPSTICK, U6 TMC2209_SILENTSTEPSTICK, U7 TMC2209_SILENTSTEPSTICK

Commit message: Adding the MTL Schematics in post editing
Other:
- note added: "The DIAG pins are necessary if you wish to use the StallGuard feedback from the TMC2209. To implement this, use the pin that sticks off the top of the module and a jumper wire and connect to GPIO pins to sense input. I recommend and is currently implemented on prototype: U5: GPIO_1 U6: GPIO_2 U7: GPIO_7"
Changed lines of the file:
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@@
+		)
+	)
+	(text "The DIAG pins are necessary if you wish to use\nthe StallGuard feedback from the TMC2209. To \nimplement this, use the pin that sticks off the top \nof the module and a jumper wire and connect to \nGPIO pins to sense input. I recommend and is currently \nimplemented on prototype: \nU5: GPIO_1\nU6: GPIO_2\nU7: GPIO_7"
+		(exclude_from_sim no)
+		(at 181.102 58.928 0)
+		(effects
+			(font
+				(size 1.27 1.27)
+			)
 		)
 	)
