File: Schematics/MotorTotem_Rev1/MotorTotem_Rev1/MotorTotem_Rev1.kicad_sch (KiCad schematic)
At the start: 14 parts, among them J10 Conn_01x03, J5 Screw_Terminal_01x02, J8 Conn_02x05_Odd_Even, J9 Conn_02x03_Odd_Even, U2 ESP32-S3-DEVKITC-1-N8R8

Commit message: Computer Vision Module Alterations
Other:
- note added: "In next version, this jumper needs to be mirrored, currently it is backwards in reference to the TagConnect cable header"
Changed lines of the file:
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@@
+		)
+	)
+	(text "In next version, this jumper needs to be mirrored, currently it is backwards in reference\nto the TagConnect cable header"
+		(exclude_from_sim no)
+		(at 188.976 139.954 0)
+		(effects
+			(font
+				(size 1.27 1.27)
+			)
 		)
 	)
