File: Schematics/MainTotem_Rev1/40P_CONN.kicad_sch (KiCad schematic)
At the start: 28 parts, among them J6 DF40C-40DS-0.4V_51_

Commit message: Layout Edits for Mezzanine Connector routing
Parts:
- removed H12: MountingHole, symbol Mechanical:MountingHole
- H10, H11, H9: footprint (none) -> MountingHole:MountingHole_3.2mm_M3_Pad_TopOnly
- J6: footprint DF40C-40DS-0.4V_51_:HIROSE_DF40C-40DS-0.4V_51_ -> 40pinMezzanineConnMale:HIROSE_DF40C-40DS-0.4V_51_
- R23, R24, R25, R26, R27, R28, R29, R30, R31, R32, R33, R34, R35, R36, R37, R38, R39, R40, R41, R42, R43, R44, R45: footprint (none) -> Resistor_SMD:R_0603_1608Metric_Pad0.98x0.95mm_HandSolder
Connections:
- net ETH_RMII_CRS_DV: now also J6.32; no longer J6.14
- net ETH_RMII_MDIO: now also J6.30; no longer J6.18
- net ETH_RMII_RXD0: now also J6.34; no longer J6.12
- net ETH_RMII_RXD1: now also J6.38; no longer J6.10
- net I2C1_SCL: now also J6.18; no longer J6.30
- net I2C1_SDA: now also J6.14; no longer J6.32
- net at J6.22: now also R41.2; no longer R38.2
- net at J6.28: now also R38.2; no longer R41.2
- net at R42.2: now also J6.12; no longer J6.34
- net at R43.2: now also J6.10; no longer J6.38
- net at J6.40: now also R37.2; no longer R45.2
- net at J6.8: now also R45.2; no longer R37.2
