File: Schematics/MainTotem_Rev1/QSPIMEM.kicad_sch (KiCad schematic)
At the start: 3 parts, among them U8 W25Q128JVSIQ TR

Commit message: Layout Edits for Mezzanine Connector routing
Parts:
- added R57: 33, Resistor_SMD:R_0603_1608Metric_Pad0.98x0.95mm_HandSolder, symbol Device:R
- C63: value C -> 100n; footprint (none) -> Capacitor_SMD:C_0603_1608Metric_Pad1.08x0.95mm_HandSolder
- R16: footprint (none) -> Resistor_SMD:R_0603_1608Metric_Pad0.98x0.95mm_HandSolder
- U8: footprint SOIC_208MIL_WIN -> MemoryChipQSPI:SOIC_208MIL_WIN-M
Connections:
- net QUADSPI_BK1_CLK: now also R57.1; no longer U8.6 (CLK)
- new net: R57.2, U8.6 (CLK)
Changed lines of the file:
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@@
-	(wire
-		(pts
-			(xy 201.93 99.06) (xy 201.93 86.36)
-		)
-		(stroke
-			(width 0)
-			(type default)
-		)
-	)
 	(wire
 		(pts
@@
 	(wire
 		(pts
+			(xy 201.93 85.09) (xy 201.93 99.06)
+		)
+		(stroke
+			(width 0)
+			(type default)
+		)
+	)
+	(wire
+		(pts
 			(xy 186.69 71.12) (xy 186.69 72.39)
 		)
@@
 		(pts
 			(xy 186.69 101.6) (xy 208.28 101.6)
+		)
+		(stroke
+			(width 0)
+			(type default)
+		)
+	)
+	(wire
+		(pts
+			(xy 201.93 72.39) (xy 201.93 77.47)
 		)
 		(stroke
@@
 	(hierarchical_label "QUADSPI_BK1_CLK"
 		(shape bidirectional)
-		(at 201.93 86.36 90)
+		(at 201.93 72.39 90)
 		(effects
 			(font
@@
 			)
 		)
-		(property "Value" "C"
+		(property "Value" "100n"
 			(at 181.61 78.7399 0)
 			(effects
@@
 			)
 		)
-		(property "Footprint" ""
+		(property "Footprint" "Capacitor_SMD:C_0603_1608Metric_Pad1.08x0.95mm_HandSolder"
 			(at 178.7652 81.28 0)
 			(effects
@@
 			)
 		)
-		(property "Footprint" "SOIC_208MIL_WIN"
+		(property "Footprint" "MemoryChipQSPI:SOIC_208MIL_WIN-M"
 			(at 105.41 93.98 0)
 			(effects
@@
 			)
 		)
-		(property "Footprint" ""
+		(property "Footprint" "Resistor_SMD:R_0603_1608Metric_Pad0.98x0.95mm_HandSolder"
 			(at 109.22 80.518 90)
 			(effects
@@
 					(unit 1)
 				)
+			)
+		)
+	)
+	(symbol
+		(lib_id "Device:R")
+		(at 201.93 81.28 0)
+		(unit 1)
+		(exclude_from_sim no)
+		(in_bom yes)
+		(on_board yes)
+		(dnp no)
+		(fields_autoplaced yes)
+		(property "Reference" "R57"
+			(at 204.47 80.0099 0)
+			(effects
+				(font
+					(size 1.27 1.27)
+				)
+				(justify left)
+			)
+		)
+		(property "Value" "33"
+			(at 204.47 82.5499 0)
+			(effects
+				(font
+					(size 1.27 1.27)
+				)
+				(justify left)
+			)
+		)
+		(property "Footprint" "Resistor_SMD:R_0603_1608Metric_Pad0.98x0.95mm_HandSolder"
+			(at 200.152 81.28 90)
+			(effects
+				(font
+					(size 1.27 1.27)
+				)
+				(hide yes)
+			)
+		)
+		(property "Datasheet" "~"
+			(at 201.93 81.28 0)
+			(effects
+				(font
+					(size 1.27 1.27)
+				)
+				(hide yes)
+			)
+		)
+		(property "Description" "Resistor"
+			(at 201.93 81.28 0)
+			(effects
+				(font
+					(size 1.27 1.27)
+				)
+				(hide yes)
+			)
+		)
+		(pin "2"
+		)
+		(pin "1"
+		)
+		(instances
+			(project ""
+				(path "/f88ba0f4-041f-4cf3-b904-3ea5c6101abb/39b009e0-d9eb-493f-99f5-9b2cb61eab22/2e64514f-165d-4acf-ba3a-af0efce37140"
+					(reference "R57")
+					(unit 1)
+				)
