File: Schematics/MainTotem_Rev1/clock.kicad_sch (KiCad schematic)
At the start: 6 parts

Commit message: Layout Edits for Mezzanine Connector routing
Parts:
- C59, C60, C61, C62: footprint (none) -> Capacitor_SMD:C_0603_1608Metric_Pad1.08x0.95mm_HandSolder
- renumbered MainClock to MainClock1, RTC to RTC1
Changed lines of the file:
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@@
 			)
 		)
-		(property "Footprint" ""
+		(property "Footprint" "Capacitor_SMD:C_0603_1608Metric_Pad1.08x0.95mm_HandSolder"
 			(at 126.6952 118.11 0)
 			(effects
@@
 			)
 		)
-		(property "Footprint" ""
+		(property "Footprint" "Capacitor_SMD:C_0603_1608Metric_Pad1.08x0.95mm_HandSolder"
 			(at 131.7752 63.5 0)
 			(effects
@@
 		(dnp no)
 		(fields_autoplaced yes)
-		(property "Reference" "MainClock"
+		(property "Reference" "MainClock1"
 			(at 143.51 100.33 0)
 			(effects
@@
 			(project ""
 				(path "/f88ba0f4-041f-4cf3-b904-3ea5c6101abb/19d6abdf-8015-4fd4-afe9-8598d45d6109"
-					(reference "MainClock")
+					(reference "MainClock1")
 					(unit 1)
 				)
@@
 			)
 		)
-		(property "Footprint" ""
+		(property "Footprint" "Capacitor_SMD:C_0603_1608Metric_Pad1.08x0.95mm_HandSolder"
 			(at 158.4452 118.11 0)
 			(effects
@@
 			)
 		)
-		(property "Footprint" ""
+		(property "Footprint" "Capacitor_SMD:C_0603_1608Metric_Pad1.08x0.95mm_HandSolder"
 			(at 155.9052 63.5 0)
 			(effects
@@
 		(dnp no)
 		(fields_autoplaced yes)
-		(property "Reference" "RTC"
+		(property "Reference" "RTC1"
 			(at 143.51 48.26 0)
 			(effects
@@
 			(project ""
 				(path "/f88ba0f4-041f-4cf3-b904-3ea5c6101abb/19d6abdf-8015-4fd4-afe9-8598d45d6109"
-					(reference "RTC")
-					(unit 1)
-				)
+					(reference "RTC1")
+					(unit 1)
+				)
