File: Schematics/MainTotem_Rev1/ShamanLinkPower.kicad_sch (KiCad schematic)
At the start: 11 parts, among them U11 PTPS2117DRLR

Commit message: Layout Edits for Mezzanine Connector routing
Parts:
- 3V3: footprint (none) -> TestPoint:TestPoint_Pad_1.0x1.0mm
- C72, C73, C74, C75, C76: footprint (none) -> Capacitor_SMD:C_0603_1608Metric_Pad1.08x0.95mm_HandSolder
- C77: footprint (none) -> Capacitor_SMD:C_0805_2012Metric_Pad1.18x1.45mm_HandSolder
- R19, R20, R21: footprint (none) -> Resistor_SMD:R_0603_1608Metric_Pad0.98x0.95mm_HandSolder
- U11: footprint SOT-5X3-8_DRL_TEX -> TPS2117:SOT-5X3-8_DRL_TEX-M
Changed lines of the file:
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@@
 			)
 		)
-		(property "Footprint" ""
+		(property "Footprint" "TestPoint:TestPoint_Pad_1.0x1.0mm"
 			(at 243.84 85.09 0)
 			(effects
@@
 			)
 		)
-		(property "Footprint" ""
+		(property "Footprint" "Capacitor_SMD:C_0603_1608Metric_Pad1.08x0.95mm_HandSolder"
 			(at 149.5552 140.97 0)
 			(effects
@@
 			)
 		)
-		(property "Footprint" ""
+		(property "Footprint" "Capacitor_SMD:C_0805_2012Metric_Pad1.18x1.45mm_HandSolder"
 			(at 249.8852 107.95 0)
 			(effects
@@
 			)
 		)
-		(property "Footprint" ""
+		(property "Footprint" "Capacitor_SMD:C_0603_1608Metric_Pad1.08x0.95mm_HandSolder"
 			(at 238.4552 107.95 0)
 			(effects
@@
 			)
 		)
-		(property "Footprint" ""
+		(property "Footprint" "Capacitor_SMD:C_0603_1608Metric_Pad1.08x0.95mm_HandSolder"
 			(at 215.5952 110.49 0)
 			(effects
@@
 			)
 		)
-		(property "Footprint" ""
+		(property "Footprint" "Capacitor_SMD:C_0603_1608Metric_Pad1.08x0.95mm_HandSolder"
 			(at 227.0252 110.49 0)
 			(effects
@@
 			)
 		)
-		(property "Footprint" ""
+		(property "Footprint" "Resistor_SMD:R_0603_1608Metric_Pad0.98x0.95mm_HandSolder"
 			(at 209.042 93.98 90)
 			(effects
@@
 			)
 		)
-		(property "Footprint" ""
+		(property "Footprint" "Resistor_SMD:R_0603_1608Metric_Pad0.98x0.95mm_HandSolder"
 			(at 166.37 107.188 90)
 			(effects
@@
 			)
 		)
-		(property "Footprint" ""
+		(property "Footprint" "Capacitor_SMD:C_0603_1608Metric_Pad1.08x0.95mm_HandSolder"
 			(at 160.9852 140.97 0)
 			(effects
@@
 			)
 		)
-		(property "Footprint" "SOT-5X3-8_DRL_TEX"
+		(property "Footprint" "TPS2117:SOT-5X3-8_DRL_TEX-M"
 			(at 170.18 97.79 0)
 			(effects
@@
 			)
 		)
-		(property "Footprint" ""
+		(property "Footprint" "Resistor_SMD:R_0603_1608Metric_Pad0.98x0.95mm_HandSolder"
 			(at 168.402 109.22 90)
 			(effects

Commit message: Computer Vision Module Alterations
Connections:
- net 3V3MODULES: now also C72.1, C73.1, R19.1, R21.1, U11.3 (VIN1), U11.5 (MODE); no longer C74.1, C75.1, U11.6 (VIN2)
- net 3V3PROGRAMMER: now also C74.1, C75.1, U11.6 (VIN2); no longer C72.1, C73.1, R19.1, R21.1, U11.3 (VIN1), U11.5 (MODE)
Changed lines of the file:
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@@
-	(wire
-		(pts
-			(xy 228.6 59.69) (xy 228.6 102.87)
-		)
-		(stroke
-			(width 0)
-			(type default)
-		)
-	)
 	(wire
 		(pts
@@
 	(wire
 		(pts
+			(xy 129.54 58.42) (xy 228.6 58.42)
+		)
+		(stroke
+			(width 0)
+			(type default)
+		)
+	)
+	(wire
+		(pts
 			(xy 248.92 85.09) (xy 248.92 100.33)
 		)
@@
 	(wire
 		(pts
-			(xy 133.35 59.69) (xy 228.6 59.69)
-		)
-		(stroke
-			(width 0)
-			(type default)
-		)
-	)
-	(wire
-		(pts
 			(xy 144.78 105.41) (xy 162.56 105.41)
 		)
@@
 	(wire
 		(pts
+			(xy 107.95 102.87) (xy 144.78 102.87)
+		)
+		(stroke
+			(width 0)
+			(type default)
+		)
+	)
+	(wire
+		(pts
 			(xy 238.76 85.09) (xy 248.92 85.09)
 		)
@@
 	(wire
 		(pts
+			(xy 228.6 58.42) (xy 228.6 102.87)
+		)
+		(stroke
+			(width 0)
+			(type default)
+		)
+	)
+	(wire
+		(pts
 			(xy 248.92 100.33) (xy 237.49 100.33)
 		)
@@
 		(pts
 			(xy 144.78 102.87) (xy 170.18 102.87)
-		)
-		(stroke
-			(width 0)
-			(type default)
-		)
-	)
-	(wire
-		(pts
-			(xy 130.81 102.87) (xy 144.78 102.87)
 		)
 		(stroke
@@
 	(global_label "3V3PROGRAMMER"
 		(shape bidirectional)
-		(at 130.81 102.87 180)
+		(at 129.54 58.42 180)
 		(fields_autoplaced yes)
 		(effects
@@
 		)
 		(property "Intersheetrefs" "${INTERSHEET_REFS}"
-			(at 110.385 102.87 0)
+			(at 109.115 58.42 0)
 			(effects
 				(font
@@
 	(global_label "3V3MODULES"
 		(shape bidirectional)
-		(at 133.35 59.69 180)
+		(at 107.95 102.87 180)
 		(fields_autoplaced yes)
 		(effects
@@
 		)
 		(property "Intersheetrefs" "${INTERSHEET_REFS}"
-			(at 116.9769 59.69 0)
+			(at 91.5769 102.87 0)
 			(effects
 				(font
