File: Schematics/MainTotem_Rev1/MainTotem_Rev1.kicad_pcb (KiCad board)
At the start: 2 copper layers, 1 part, among them U1 STM32H757IIT6

Commit message: Layout Edits for Mezzanine Connector routing
Parts:
- added 3V3: TestPoint, TestPoint:TestPoint_Pad_1.0x1.0mm, F.Cu at (158.8, 101.4)
- added 3V3HPSoC: YELLOW, Resistor_SMD:R_0805_2012Metric_Pad1.20x1.40mm_HandSolder, F.Cu at (174.6, 95.0)
- added 3V3HSSoC: GREEN, Resistor_SMD:R_0805_2012Metric_Pad1.20x1.40mm_HandSolder, F.Cu at (172.4, 114.0)
- added 3V3SoC: TestPoint, TestPoint:TestPoint_Pad_1.0x1.0mm, F.Cu at (173.4, 107.0)
- added C1: 100n, Capacitor_SMD:C_0603_1608Metric_Pad1.08x0.95mm_HandSolder, F.Cu at (145.7, 100.2)
- added C10: 100n, Capacitor_SMD:C_0603_1608Metric_Pad1.08x0.95mm_HandSolder, F.Cu at (156.8, 67.6)
- added C11: 100n, Capacitor_SMD:C_0603_1608Metric_Pad1.08x0.95mm_HandSolder, F.Cu at (158.9, 69.7)
- added C12: 100n, Capacitor_SMD:C_0603_1608Metric_Pad1.08x0.95mm_HandSolder, F.Cu at (164.8, 75.4)
- added C13: 100n, Capacitor_SMD:C_0603_1608Metric_Pad1.08x0.95mm_HandSolder, B.Cu at (159.7, 89.6)
- added C14: 100n, Capacitor_SMD:C_0603_1608Metric_Pad1.08x0.95mm_HandSolder, B.Cu at (153.7, 92.0)
- added C15: 100n, Capacitor_SMD:C_0603_1608Metric_Pad1.08x0.95mm_HandSolder, F.Cu at (166.3, 82.1)
- added C16: 100n, Capacitor_SMD:C_0603_1608Metric_Pad1.08x0.95mm_HandSolder, F.Cu at (149.0, 100.5)
- added C17: 4.7u, Capacitor_SMD:C_0603_1608Metric_Pad1.08x0.95mm_HandSolder, B.Cu at (146.2, 68.2)
- added C18: 1u, Capacitor_SMD:C_0603_1608Metric_Pad1.08x0.95mm_HandSolder, B.Cu at (160.0, 79.6)
- added C19: 100n, Capacitor_SMD:C_0603_1608Metric_Pad1.08x0.95mm_HandSolder, B.Cu at (161.1, 80.6)
- added C2: 100n, Capacitor_SMD:C_0603_1608Metric_Pad1.08x0.95mm_HandSolder, F.Cu at (137.6, 93.1)
- added C20: 1u, Capacitor_SMD:C_0603_1608Metric_Pad1.08x0.95mm_HandSolder, B.Cu at (166.9, 85.8)
- added C21: 100n, Capacitor_SMD:C_0603_1608Metric_Pad1.08x0.95mm_HandSolder, B.Cu at (164.7, 86.2)
- added C22: 100n, Capacitor_SMD:C_0603_1608Metric_Pad1.08x0.95mm_HandSolder, B.Cu at (174.3, 77.7)
- added C23: 0.1u, Capacitor_SMD:C_0603_1608Metric_Pad1.08x0.95mm_HandSolder, F.Cu at (198.3, 89.3)
- added C24: 10u, Capacitor_SMD:C_0805_2012Metric_Pad1.18x1.45mm_HandSolder, F.Cu at (87.8, 84.0)
- added C25: 0.1u, Capacitor_SMD:C_0603_1608Metric_Pad1.08x0.95mm_HandSolder, F.Cu at (91.9, 84.9)
- added C26: 100n, Capacitor_SMD:C_0603_1608Metric_Pad1.08x0.95mm_HandSolder, F.Cu at (165.8, 85.2)
- added C27: 100n, Capacitor_SMD:C_0603_1608Metric_Pad1.08x0.95mm_HandSolder, F.Cu at (96.8, 63.0)
- added C28: 2.2u ESR<100m, Capacitor_SMD:C_0603_1608Metric_Pad1.08x0.95mm_HandSolder, F.Cu at (141.7, 97.8)
- added C29: 2.2u ESR<100m, Capacitor_SMD:C_0603_1608Metric_Pad1.08x0.95mm_HandSolder, F.Cu at (127.8, 82.0)
- added C3: 100n, Capacitor_SMD:C_0603_1608Metric_Pad1.08x0.95mm_HandSolder, F.Cu at (134.8, 90.3)
- added C30: 2.2u ESR<100m, Capacitor_SMD:C_0603_1608Metric_Pad1.08x0.95mm_HandSolder, B.Cu at (149.2, 68.4)
- added C31: 2.2u ESR<100m, Capacitor_SMD:C_0603_1608Metric_Pad1.08x0.95mm_HandSolder, F.Cu at (138.6, 66.0)
- added C32: 100n, Capacitor_SMD:C_0603_1608Metric_Pad1.08x0.95mm_HandSolder, B.Cu at (101.0, 67.9)
- added C33: 10u, Capacitor_SMD:C_0805_2012Metric_Pad1.18x1.45mm_HandSolder, F.Cu at (190.1, 90.8)
- added C34: 100n, Capacitor_SMD:C_0603_1608Metric_Pad1.08x0.95mm_HandSolder, F.Cu at (188.3, 86.3)
- added C35: 100n, Capacitor_SMD:C_0603_1608Metric_Pad1.08x0.95mm_HandSolder, F.Cu at (182.2, 89.2)
- added C36: 10u, Capacitor_SMD:C_0805_2012Metric_Pad1.18x1.45mm_HandSolder, F.Cu at (181.9, 94.0)
- added C37: 10u, Capacitor_SMD:C_0805_2012Metric_Pad1.18x1.45mm_HandSolder, F.Cu at (163.7, 105.4)
- added C38: 100n, Capacitor_SMD:C_0603_1608Metric_Pad1.08x0.95mm_HandSolder, F.Cu at (159.2, 107.0)
- added C39: 100n, Capacitor_SMD:C_0603_1608Metric_Pad1.08x0.95mm_HandSolder, F.Cu at (162.2, 113.2)
- added C4: 100n, Capacitor_SMD:C_0603_1608Metric_Pad1.08x0.95mm_HandSolder, B.Cu at (133.1, 80.7)
- added C40: 10u, Capacitor_SMD:C_0805_2012Metric_Pad1.18x1.45mm_HandSolder, F.Cu at (168.3, 112.9)
- added C41: 4.7u, Capacitor_SMD:C_0603_1608Metric_Pad1.08x0.95mm_HandSolder, F.Cu at (176.2, 105.6)
- added C42: 0.1u, Capacitor_SMD:C_0603_1608Metric_Pad1.08x0.95mm_HandSolder, F.Cu at (178.0, 105.1)
- added C43: 4.7u, Capacitor_SMD:C_0603_1608Metric_Pad1.08x0.95mm_HandSolder, F.Cu at (179.9, 96.5)
- added C44: 0.1u, Capacitor_SMD:C_0603_1608Metric_Pad1.08x0.95mm_HandSolder, F.Cu at (178.5, 98.0)
- added C45: 0.1u, Capacitor_SMD:C_0603_1608Metric_Pad1.08x0.95mm_HandSolder, B.Cu at (177.4, 103.3)
- added C46: 22u, Capacitor_SMD:C_0805_2012Metric_Pad1.18x1.45mm_HandSolder, B.Cu at (175.4, 106.4)
- added C47: 100n, Capacitor_SMD:C_0603_1608Metric_Pad1.08x0.95mm_HandSolder, F.Cu at (143.0, 99.1)
- added C48: 100n, Capacitor_SMD:C_0603_1608Metric_Pad1.08x0.95mm_HandSolder, F.Cu at (128.5, 85.0)
- added C49: 100n, Capacitor_SMD:C_0603_1608Metric_Pad1.08x0.95mm_HandSolder, F.Cu at (153.2, 63.0)
- added C5: 100n, Capacitor_SMD:C_0603_1608Metric_Pad1.08x0.95mm_HandSolder, B.Cu at (134.7, 78.6)
- added C51: 100n, Capacitor_SMD:C_0603_1608Metric_Pad1.08x0.95mm_HandSolder, F.Cu at (151.1, 98.3)
- added C52: 100n, Capacitor_SMD:C_0603_1608Metric_Pad1.08x0.95mm_HandSolder, F.Cu at (137.3, 67.2)
- added C54: 100n, Capacitor_SMD:C_0603_1608Metric_Pad1.08x0.95mm_HandSolder, F.Cu at (132.1, 72.4)
- added C55: 4.7u ESR<100m, Capacitor_SMD:C_0603_1608Metric_Pad1.08x0.95mm_HandSolder, F.Cu at (156.5, 92.9)
- added C56: 220pF, Capacitor_SMD:C_0603_1608Metric_Pad1.08x0.95mm_HandSolder, F.Cu at (156.4, 94.4)
- added C57: 10u ESR<20m, Capacitor_SMD:C_0805_2012Metric_Pad1.18x1.45mm_HandSolder, F.Cu at (159.8, 96.4)
- added C58: 10u ESR<20m, Capacitor_SMD:C_0805_2012Metric_Pad1.18x1.45mm_HandSolder, F.Cu at (160.1, 93.3)
- added C59: 12p, Capacitor_SMD:C_0603_1608Metric_Pad1.08x0.95mm_HandSolder, F.Cu at (163.5, 87.1)
- added C6: 100n, Capacitor_SMD:C_0603_1608Metric_Pad1.08x0.95mm_HandSolder, F.Cu at (135.1, 69.6)
- added C60: 12p, Capacitor_SMD:C_0603_1608Metric_Pad1.08x0.95mm_HandSolder, F.Cu at (160.9, 89.3)
- added C61: 15p, Capacitor_SMD:C_0603_1608Metric_Pad1.08x0.95mm_HandSolder, F.Cu at (154.8, 96.9)
- added C62: 15p, Capacitor_SMD:C_0603_1608Metric_Pad1.08x0.95mm_HandSolder, F.Cu at (153.1, 96.6)
- added C63: 100n, Capacitor_SMD:C_0603_1608Metric_Pad1.08x0.95mm_HandSolder, B.Cu at (147.6, 88.2)
- added C64: 0.1u, Capacitor_SMD:C_0603_1608Metric_Pad1.08x0.95mm_HandSolder, F.Cu at (80.6, 75.0)
- added C7: 100n, Capacitor_SMD:C_0603_1608Metric_Pad1.08x0.95mm_HandSolder, F.Cu at (139.8, 64.8)
- added C72: 4.7u, Capacitor_SMD:C_0603_1608Metric_Pad1.08x0.95mm_HandSolder, F.Cu at (162.2, 101.4)
- added C73: 0.1u, Capacitor_SMD:C_0603_1608Metric_Pad1.08x0.95mm_HandSolder, F.Cu at (164.4, 101.5)
- added C74: 4.7u, Capacitor_SMD:C_0603_1608Metric_Pad1.08x0.95mm_HandSolder, F.Cu at (172.0, 104.4)
- added C75: 0.1u, Capacitor_SMD:C_0603_1608Metric_Pad1.08x0.95mm_HandSolder, F.Cu at (171.1, 101.7)
- added C76: 0.1u, Capacitor_SMD:C_0603_1608Metric_Pad1.08x0.95mm_HandSolder, B.Cu at (166.3, 97.5)
- added C77: 22u, Capacitor_SMD:C_0805_2012Metric_Pad1.18x1.45mm_HandSolder, B.Cu at (172.4, 97.4)
- added C8: 100n, Capacitor_SMD:C_0603_1608Metric_Pad1.08x0.95mm_HandSolder, F.Cu at (142.1, 62.5)
- added C9: 100n, Capacitor_SMD:C_0603_1608Metric_Pad1.08x0.95mm_HandSolder, F.Cu at (151.6, 62.2)
- added D1: SM712_SOT23, Package_TO_SOT_SMD:SOT-23, F.Cu at (82.2, 79.7)
- added D2: GREEN, Resistor_SMD:R_0805_2012Metric_Pad1.20x1.40mm_HandSolder, F.Cu at (126.0, 66.0)
- added D3: YELLOW, Resistor_SMD:R_0805_2012Metric_Pad1.20x1.40mm_HandSolder, F.Cu at (124.2, 67.9)
- added D4: BAT54SW_115, BAT54SW_115:BAT54SW_115, F.Cu at (168.1, 89.6)
- added D6: RED, Resistor_SMD:R_0805_2012Metric_Pad1.20x1.40mm_HandSolder, F.Cu at (127.8, 64.1)
- added FB1: MFBW1V1608-601-R, Resistor_SMD:R_0603_1608Metric_Pad0.98x0.95mm_HandSolder, B.Cu at (158.9, 78.4)
- added G***: LOGO, MakeyDooeyLogo:MakeyDooeyLogo, F.Cu at (107.8, 58.3)
- added GND: TestPoint, TestPoint:TestPoint_Pad_1.0x1.0mm, F.Cu at (173.4, 110.5)
- added H1: MountingHole, MountingHole:MountingHole_3.2mm_M3_Pad_TopOnly, F.Cu at (83.8, 54.6)
- added H10: MountingHole, MountingHole:MountingHole_3.2mm_M3_Pad_TopOnly, F.Cu at (122.7, 88.0)
- added H11: MountingHole, MountingHole:MountingHole_3.2mm_M3_Pad_TopOnly, F.Cu at (142.2, 110.6)
- added H2: MountingHole, MountingHole:MountingHole_3.2mm_M3_Pad_TopOnly, F.Cu at (194.8, 54.7)
- added H3: MountingHole, MountingHole:MountingHole_3.2mm_M3_Pad_TopOnly, F.Cu at (84.2, 115.7)
- added H4: MountingHole, MountingHole:MountingHole_3.2mm_M3_Pad_TopOnly, F.Cu at (195.6, 113.3)
- added H5: MountingHole, MountingHole:MountingHole_3.2mm_M3_Pad_TopOnly, F.Cu at (186.0, 54.8)
- added H7: MountingHole, MountingHole:MountingHole_3.2mm_M3_Pad_TopOnly, F.Cu at (186.4, 80.9)
- added H7RST1: SW_Push, Button_Switch_SMD:SW_SPST_PTS645Sx43SMTR92, F.Cu at (174.8, 90.3)
- added H7_UART/SWD: Conn_02x05_Odd_Even, Connector_PinHeader_2.54mm:PinHeader_2x05_P2.54mm_Vertical, F.Cu at (95.9, 92.4)
- added H8: MountingHole, MountingHole:MountingHole_3.2mm_M3_Pad_TopOnly, F.Cu at (136.2, 55.6)
- added H9: MountingHole, MountingHole:MountingHole_3.2mm_M3_Pad_TopOnly, F.Cu at (99.9, 110.5)
- added J1: S6B-XH-A, JSTS6B-XH-A-1:JST_S6B-XH-A, F.Cu at (207.5, 82.1)
- added J2: S6B-XH-A, JSTS6B-XH-A-1:JST_S6B-XH-A, F.Cu at (71.4, 82.3)
- added J3: Conn_02x05_Odd_Even, Connector_PinHeader_2.54mm:PinHeader_2x05_P2.54mm_Vertical, F.Cu at (89.1, 66.6)
- added J5: DF40C-100DS-0.4V_51_, 100pinMezzanineConnMale:HIROSE_DF40C-100DS-0.4V_51_, F.Cu at (177.3, 62.7)
- added J6: DF40C-40DS-0.4V_51_, 40pinMezzanineConnMale:HIROSE_DF40C-40DS-0.4V_51_, F.Cu at (111.6, 110.7)
- added JP1: Jumper_2_Open, Connector_PinHeader_2.54mm:PinHeader_1x02_P2.54mm_Vertical, F.Cu at (86.6, 75.6)
- added L1: VLS252012CX-2R2M-1, 22uFInductor:IND_VLS252012CX-2R2M-1, F.Cu at (157.2, 96.4)
- added MainClock1: ABM10W-24.0000MHZ-8-D1X-T3, ABM10W-24.0000MHZ-8-D1X-T3:XTAL_ABM10W-24.0000MHZ-8-D1X-T3, F.Cu at (163.5, 89.9)
- added PROG1: GREEN, Resistor_SMD:R_0805_2012Metric_Pad1.20x1.40mm_HandSolder, F.Cu at (91.7, 75.6)
- added R1: 120, Resistor_SMD:R_1210_3225Metric_Pad1.30x2.65mm_HandSolder, F.Cu at (87.3, 80.0)
- added R10: 1k, Resistor_SMD:R_0603_1608Metric_Pad0.98x0.95mm_HandSolder, B.Cu at (95.8, 76.8)
- added R11: 1k, Resistor_SMD:R_0603_1608Metric_Pad0.98x0.95mm_HandSolder, F.Cu at (178.6, 94.9)
- added R12: 1k, Resistor_SMD:R_0603_1608Metric_Pad0.98x0.95mm_HandSolder, F.Cu at (170.2, 110.8)
- added R13: 56k, Resistor_SMD:R_0603_1608Metric_Pad0.98x0.95mm_HandSolder, F.Cu at (180.7, 101.5)
- added R14: 110k, Resistor_SMD:R_0603_1608Metric_Pad0.98x0.95mm_HandSolder, F.Cu at (180.2, 103.5)
- added R15: 100k, Resistor_SMD:R_0603_1608Metric_Pad0.98x0.95mm_HandSolder, F.Cu at (174.3, 100.9)
- added R16: 10k, Resistor_SMD:R_0603_1608Metric_Pad0.98x0.95mm_HandSolder, B.Cu at (150.4, 76.1)
- added R17: 1k, Resistor_SMD:R_0603_1608Metric_Pad0.98x0.95mm_HandSolder, F.Cu at (123.8, 62.3)
- added R18: 1k, Resistor_SMD:R_0603_1608Metric_Pad0.98x0.95mm_HandSolder, F.Cu at (121.5, 64.2)
- added R19: 110k, Resistor_SMD:R_0603_1608Metric_Pad0.98x0.95mm_HandSolder, F.Cu at (166.8, 102.7)
- added R2: 10k, Resistor_SMD:R_0603_1608Metric_Pad0.98x0.95mm_HandSolder, F.Cu at (99.5, 82.9)
- added R20: 56k, Resistor_SMD:R_0603_1608Metric_Pad0.98x0.95mm_HandSolder, F.Cu at (169.3, 103.6)
- added R21: 100k, Resistor_SMD:R_0603_1608Metric_Pad0.98x0.95mm_HandSolder, F.Cu at (168.3, 97.2)
- added R22: 1k, Resistor_SMD:R_0603_1608Metric_Pad0.98x0.95mm_HandSolder, F.Cu at (119.7, 66.3)
- added R23: 4.7k, Resistor_SMD:R_0603_1608Metric_Pad0.98x0.95mm_HandSolder, F.Cu at (127.3, 111.5)
- added R24: 4.7k, Resistor_SMD:R_0603_1608Metric_Pad0.98x0.95mm_HandSolder, F.Cu at (123.9, 114.9)
- added R25: 10k, Resistor_SMD:R_0603_1608Metric_Pad0.98x0.95mm_HandSolder, F.Cu at (115.9, 106.1)
- added R26: 10k, Resistor_SMD:R_0603_1608Metric_Pad0.98x0.95mm_HandSolder, F.Cu at (114.8, 102.6)
- added R27: 10k, Resistor_SMD:R_0603_1608Metric_Pad0.98x0.95mm_HandSolder, F.Cu at (117.5, 98.5)
- added R28: 10k, Resistor_SMD:R_0603_1608Metric_Pad0.98x0.95mm_HandSolder, F.Cu at (115.9, 93.4)
- added R29: 10k, Resistor_SMD:R_0603_1608Metric_Pad0.98x0.95mm_HandSolder, F.Cu at (114.2, 91.8)
- added R3: 10k, Resistor_SMD:R_0603_1608Metric_Pad0.98x0.95mm_HandSolder, F.Cu at (99.5, 78.9)
- added R30: 33, Resistor_SMD:R_0603_1608Metric_Pad0.98x0.95mm_HandSolder, F.Cu at (129.8, 88.0)
- added R31: 10k, Resistor_SMD:R_0603_1608Metric_Pad0.98x0.95mm_HandSolder, F.Cu at (126.0, 100.7)
- added R32: 10k, Resistor_SMD:R_0603_1608Metric_Pad0.98x0.95mm_HandSolder, F.Cu at (120.6, 101.9)
- added R33: 33, Resistor_SMD:R_0603_1608Metric_Pad0.98x0.95mm_HandSolder, F.Cu at (129.5, 93.0)
- added R34: 33, Resistor_SMD:R_0603_1608Metric_Pad0.98x0.95mm_HandSolder, F.Cu at (127.7, 96.2)
- added R35: 33, Resistor_SMD:R_0603_1608Metric_Pad0.98x0.95mm_HandSolder, F.Cu at (131.1, 94.4)
- added R36: 33, Resistor_SMD:R_0603_1608Metric_Pad0.98x0.95mm_HandSolder, F.Cu at (133.7, 94.5)
- added R37: 33, Resistor_SMD:R_0603_1608Metric_Pad0.98x0.95mm_HandSolder, F.Cu at (134.7, 96.5)
- added R38: 33, Resistor_SMD:R_0603_1608Metric_Pad0.98x0.95mm_HandSolder, F.Cu at (138.0, 101.5)
- added R39: 33, Resistor_SMD:R_0603_1608Metric_Pad0.98x0.95mm_HandSolder, B.Cu at (150.2, 70.3)
- added R4: 10k, Resistor_SMD:R_0603_1608Metric_Pad0.98x0.95mm_HandSolder, B.Cu at (144.6, 91.6)
- added R40: 33, Resistor_SMD:R_0603_1608Metric_Pad0.98x0.95mm_HandSolder, F.Cu at (139.0, 103.0)
- added R41: 33, Resistor_SMD:R_0603_1608Metric_Pad0.98x0.95mm_HandSolder, F.Cu at (137.4, 96.2)
- added R42: 33, Resistor_SMD:R_0603_1608Metric_Pad0.98x0.95mm_HandSolder, B.Cu at (143.4, 95.7)
- added R43: 33, Resistor_SMD:R_0603_1608Metric_Pad0.98x0.95mm_HandSolder, B.Cu at (144.5, 96.8)
- added R44: 4.7k, Resistor_SMD:R_0603_1608Metric_Pad0.98x0.95mm_HandSolder, F.Cu at (119.7, 112.5)
- added R45: 33, Resistor_SMD:R_0603_1608Metric_Pad0.98x0.95mm_HandSolder, F.Cu at (139.9, 104.9)
- added R46: 33, Resistor_SMD:R_0603_1608Metric_Pad0.98x0.95mm_HandSolder, F.Cu at (207.7, 31.5)
- added R47: 33, Resistor_SMD:R_0603_1608Metric_Pad0.98x0.95mm_HandSolder, F.Cu at (207.7, 34.0)
- added R48: 10k, Resistor_SMD:R_0603_1608Metric_Pad0.98x0.95mm_HandSolder, F.Cu at (207.7, 36.5)
- added R49: 10k, Resistor_SMD:R_0603_1608Metric_Pad0.98x0.95mm_HandSolder, F.Cu at (207.7, 39.1)
- added R5: 10k, Resistor_SMD:R_0603_1608Metric_Pad0.98x0.95mm_HandSolder, F.Cu at (169.5, 86.2)
- added R50: 4.7k, Resistor_SMD:R_0603_1608Metric_Pad0.98x0.95mm_HandSolder, F.Cu at (207.7, 41.6)
- added R51: 4.7k, Resistor_SMD:R_0603_1608Metric_Pad0.98x0.95mm_HandSolder, F.Cu at (207.7, 44.1)
- added R52: 10k, Resistor_SMD:R_0603_1608Metric_Pad0.98x0.95mm_HandSolder, F.Cu at (212.1, 31.5)
- added R53: 10k, Resistor_SMD:R_0603_1608Metric_Pad0.98x0.95mm_HandSolder, F.Cu at (212.1, 34.0)
- added R54: 33, Resistor_SMD:R_0603_1608Metric_Pad0.98x0.95mm_HandSolder, F.Cu at (212.1, 36.5)
- added R55: 33, Resistor_SMD:R_0603_1608Metric_Pad0.98x0.95mm_HandSolder, F.Cu at (212.1, 39.1)
- added R56: 33, Resistor_SMD:R_0603_1608Metric_Pad0.98x0.95mm_HandSolder, F.Cu at (212.1, 41.6)
- added R57: 33, Resistor_SMD:R_0603_1608Metric_Pad0.98x0.95mm_HandSolder, B.Cu at (156.6, 82.7)
- added R6: 10k, Resistor_SMD:R_0603_1608Metric_Pad0.98x0.95mm_HandSolder, F.Cu at (124.0, 78.7)
- added R7: 10k, Resistor_SMD:R_0603_1608Metric_Pad0.98x0.95mm_HandSolder, B.Cu at (98.3, 70.4)
- added R8: 1k, Resistor_SMD:R_0603_1608Metric_Pad0.98x0.95mm_HandSolder, B.Cu at (88.8, 70.6)
- added R9: 1k, Resistor_SMD:R_0603_1608Metric_Pad0.98x0.95mm_HandSolder, B.Cu at (86.3, 70.8)
- added RN1: CAY16-330J4LF, 33ohmresistorarray:33ohmresarray, F.Cu at (208.2, 22.9)
- added RN10: CAY16-330J4LF, 33ohmresistorarray:33ohmresarray, F.Cu at (227.1, 27.8)
- added RN2: CAY16-330J4LF, 33ohmresistorarray:33ohmresarray, F.Cu at (212.9, 22.9)
- added RN3: CAY16-330J4LF, 33ohmresistorarray:33ohmresarray, F.Cu at (217.6, 22.9)
- added RN4: CAY16-330J4LF, 33ohmresistorarray:33ohmresarray, F.Cu at (222.4, 22.9)
- added RN5: CAY16-330J4LF, 33ohmresistorarray:33ohmresarray, F.Cu at (227.1, 22.9)
- added RN6: CAY16-330J4LF, 33ohmresistorarray:33ohmresarray, F.Cu at (208.2, 27.8)
- added RN7: CAY16-330J4LF, 33ohmresistorarray:33ohmresarray, F.Cu at (212.9, 27.8)
- added RN8: CAY16-330J4LF, 33ohmresistorarray:33ohmresarray, F.Cu at (217.6, 27.8)
- added RN9: CAY16-330J4LF, 33ohmresistorarray:33ohmresarray, F.Cu at (222.4, 27.8)
- added RS485: YELLOW, Resistor_SMD:R_0805_2012Metric_Pad1.20x1.40mm_HandSolder, F.Cu at (82.2, 68.3)
- added RTC1: ABS07-32.768KHZ-9-T, ABS07-32.768KHZ-9-T:XTAL_ABS07-32.768KHZ-9-T, F.Cu at (154.5, 100.0)
- added SW1: 3-1825010-8, 6PDTSwitch:SW6_3-1825010-8_TEC, F.Cu at (114.6, 73.6)
- added U11: PTPS2117DRLR, TPS2117:SOT-5X3-8_DRL_TEX-M, F.Cu at (168.3, 100.1)
- added U2: ADR4525BRZ-R7, ADR4525BRZ:R_8_ADI-M, B.Cu at (170.3, 80.9)
- added U3: THVD1450D, RS485Transceiver:D0008A_M, F.Cu at (94.1, 80.6)
- added U4: STM32G071KBT6, STM32G0:LQFP-32-M, F.Cu at (99.5, 69.4)
- added U5: AP7361C-33Y5-13, LDO_ShamanLink:SOT89-5_DIO-M, F.Cu at (185.8, 90.4)
- added U6: AP7361C-33Y5-13, LDO_ShamanLink:SOT89-5_DIO-M, F.Cu at (163.4, 109.6)
- added U7: PTPS2117DRLR, TPS2117:SOT-5X3-8_DRL_TEX-M, F.Cu at (176.9, 100.9)
- added U8: W25Q128JVSIQ TR, MemoryChipQSPI:SOIC_208MIL_WIN-M, B.Cu at (151.3, 83.1)
- added UH_OH: RED, Resistor_SMD:R_0805_2012Metric_Pad1.20x1.40mm_HandSolder, F.Cu at (82.2, 64.7)
- added USER: SW_Push, Button_Switch_SMD:SW_SPST_PTS645Sx43SMTR92, F.Cu at (152.7, 108.0)
- moved U1 21.0 mm to (147.0, 80.2), turned to 135 degrees
Connections:
- U1 pad 1: unconnected-(U1B-PE2-Pad1) -> /MCU2/100P_CONN/SAI1_MCLK
- U1 pad 10: unconnected-(U1A-PC14-OSC32_IN-Pad10) -> OSC32_IN
- U1 pad 100: unconnected-(U1C-VSS-Pad100) -> GND
- U1 pad 101: unconnected-(U1C-VCAPDSI-Pad101) -> Net-(U1C-VCAPDSI)
- U1 pad 102: unconnected-(U1C-VDD12DSI-Pad102) -> Net-(U1C-VCAPDSI)
- U1 pad 105: unconnected-(U1C-VSSDSI-Pad105) -> GND
- U1 pad 108: unconnected-(U1C-VDD12DSI-Pad108) -> Net-(U1C-VCAPDSI)
- U1 pad 109: unconnected-(U1C-VSSDSI-Pad109) -> GND
- U1 pad 11: unconnected-(U1A-PC15-OSC32_OUT-Pad11) -> OSC32_OUT
- U1 pad 110: unconnected-(U1B-PG2-Pad110) -> /MCU2/100P_CONN/GPIO_PG2
- U1 pad 111: unconnected-(U1B-PG3-Pad111) -> /MCU2/100P_CONN/GPIO_PG3
- U1 pad 112: unconnected-(U1C-VSS-Pad112) -> GND
- U1 pad 113: unconnected-(U1C-VDD-Pad113) -> +3V3
- U1 pad 114: unconnected-(U1B-PG4-Pad114) -> /MCU2/100P_CONN/GPIO_PG4
- U1 pad 115: unconnected-(U1B-PG5-Pad115) -> /MCU2/100P_CONN/GPIO_PG5
- U1 pad 116: unconnected-(U1B-PG6-Pad116) -> /MCU2/100P_CONN/GPIO_PG6
- U1 pad 117: unconnected-(U1B-PG7-Pad117) -> USART6_CTS
- U1 pad 118: unconnected-(U1B-PG8-Pad118) -> USART6_RTS
- U1 pad 119: unconnected-(U1C-VSS-Pad119) -> GND
- U1 pad 12: unconnected-(U1C-VSS-Pad12) -> GND
- U1 pad 120: unconnected-(U1C-VDD50USB-Pad120) -> +3V3
- U1 pad 121: unconnected-(U1C-VDD33USB-Pad121) -> +3V3
- U1 pad 122: unconnected-(U1A-PC6-Pad122) -> USART6_TX
- U1 pad 123: unconnected-(U1A-PC7-Pad123) -> USART6_RX
- U1 pad 124: unconnected-(U1A-PC8-Pad124) -> /MCU2/40P_CONN/SDMMC1_D0
- U1 pad 125: unconnected-(U1A-PC9-Pad125) -> /MCU2/40P_CONN/SDMMC1_D1
- U1 pad 126: unconnected-(U1C-VDD-Pad126) -> +3V3
- U1 pad 127: unconnected-(U1A-PA8-Pad127) -> /MCU2/100P_CONN/GPIO_PA8_CLKOUT
- U1 pad 128: unconnected-(U1A-PA9-Pad128) -> H7UARTTX
- U1 pad 129: unconnected-(U1A-PA10-Pad129) -> H7UARTRX
- U1 pad 13: unconnected-(U1C-VDD-Pad13) -> +3V3
- U1 pad 130: unconnected-(U1A-PA11-Pad130) -> USB_D-
- U1 pad 131: unconnected-(U1A-PA12-Pad131) -> USB_D+
- U1 pad 132: unconnected-(U1A-PA13-Pad132) -> H7SWDIO
- U1 pad 133: unconnected-(U1C-VCAP-Pad133) -> Net-(C29-Pad1)
- U1 pad 134: unconnected-(U1C-VSS-Pad134) -> GND
- U1 pad 135: unconnected-(U1C-VDDLDO-Pad135) -> Net-(U1C-VFBSMPS)
- U1 pad 136: unconnected-(U1C-VDD-Pad136) -> +3V3
- U1 pad 137: unconnected-(U1C-VSS-Pad137) -> GND
- U1 pad 138: unconnected-(U1A-PA14-Pad138) -> H7SWCLK
- U1 pad 14: unconnected-(U1C-VSSSMPS-Pad14) -> GND
- U1 pad 140: unconnected-(U1A-PC10-Pad140) -> /MCU2/40P_CONN/SDMMC1_D2
- U1 pad 141: unconnected-(U1A-PC11-Pad141) -> /MCU2/40P_CONN/SDMMC1_D3
- U1 pad 142: unconnected-(U1A-PC12-Pad142) -> /MCU2/40P_CONN/SDMMC1_CK
- U1 pad 143: unconnected-(U1A-PD0-Pad143) -> /MCU2/40P_CONN/FDCAN_RX
- U1 pad 144: unconnected-(U1A-PD1-Pad144) -> /MCU2/40P_CONN/FDCAN_TX
- U1 pad 145: unconnected-(U1A-PD2-Pad145) -> /MCU2/40P_CONN/SDMMC1_CMP
- U1 pad 146: unconnected-(U1A-PD3-Pad146) -> /MCU2/40P_CONN/USART2_CTS
- U1 pad 147: unconnected-(U1A-PD4-Pad147) -> /MCU2/40P_CONN/USART2_RTS
- U1 pad 148: unconnected-(U1A-PD5-Pad148) -> /MCU2/40P_CONN/USART2_TX
- U1 pad 149: unconnected-(U1A-PD6-Pad149) -> /MCU2/40P_CONN/USART2_RX
- U1 pad 15: unconnected-(U1C-VLXSMPS-Pad15) -> Net-(U1C-VLXSMPS)
- U1 pad 150: unconnected-(U1A-PD7-Pad150) -> /MCU2/40P_CONN/GPIO_PD7
- U1 pad 151: unconnected-(U1C-VSS-Pad151) -> GND
- U1 pad 152: unconnected-(U1C-VDD-Pad152) -> +3V3
- U1 pad 153: unconnected-(U1B-PG9-Pad153) -> Net-(D6-K)
- U1 pad 154: unconnected-(U1B-PG10-Pad154) -> Net-(D2-K)
- U1 pad 155: unconnected-(U1B-PG11-Pad155) -> Net-(D3-K)
- U1 pad 156: unconnected-(U1B-PG12-Pad156) -> Net-(U1B-PG12)
- U1 pad 157: unconnected-(U1B-PG13-Pad157) -> PG13
- U1 pad 158: unconnected-(U1B-PG14-Pad158) -> PG14
- U1 pad 159: unconnected-(U1C-VSS-Pad159) -> GND
- U1 pad 16: unconnected-(U1C-VDDSMPS-Pad16) -> +3V3
- U1 pad 160: unconnected-(U1C-VDD-Pad160) -> +3V3
- U1 pad 161: unconnected-(U1B-PG15-Pad161) -> GPIO_PG15
- U1 pad 162: unconnected-(U1A-PB3-Pad162) -> H7SWO
- U1 pad 167: unconnected-(U1B-BOOT0-Pad167) -> H7BOOT0
- U1 pad 168: unconnected-(U1A-PB8-Pad168) -> /MCU2/40P_CONN/I2C1_SCL
- U1 pad 169: unconnected-(U1A-PB9-Pad169) -> /MCU2/40P_CONN/I2C1_SDA
- U1 pad 17: unconnected-(U1C-VFBSMPS-Pad17) -> Net-(U1C-VFBSMPS)
- U1 pad 170: unconnected-(U1B-PE0-Pad170) -> /MCU2/40P_CONN/GPIO_PE0
- U1 pad 171: unconnected-(U1B-PE1-Pad171) -> /MCU2/40P_CONN/GPIO_PE1
- U1 pad 172: unconnected-(U1C-VCAP-Pad172) -> Net-(C28-Pad1)
- U1 pad 173: unconnected-(U1C-VSS-Pad173) -> GND
- U1 pad 174: unconnected-(U1B-PDR_ON-Pad174) -> +3V3
- U1 pad 175: unconnected-(U1C-VDDLDO-Pad175) -> Net-(U1C-VFBSMPS)
- U1 pad 176: unconnected-(U1C-VDD-Pad176) -> +3V3
- U1 pad 18: unconnected-(U1B-PF0-Pad18) -> /MCU2/100P_CONN/GPIO_PF0
- U1 pad 19: unconnected-(U1B-PF1-Pad19) -> /MCU2/100P_CONN/GPIO_PF1
- U1 pad 2: unconnected-(U1B-PE3-Pad2) -> /MCU2/40P_CONN/GPIO_PE3
- U1 pad 20: unconnected-(U1B-PF2-Pad20) -> /MCU2/100P_CONN/GPIO_PF2
- U1 pad 21: unconnected-(U1B-PF3-Pad21) -> /MCU2/100P_CONN/GPIO_PF3
- U1 pad 22: unconnected-(U1B-PF4-Pad22) -> /MCU2/100P_CONN/GPIO_PF4
- U1 pad 23: unconnected-(U1B-PF5-Pad23) -> /MCU2/100P_CONN/GPIO_PF5
- U1 pad 24: unconnected-(U1C-VSS-Pad24) -> GND
- U1 pad 25: unconnected-(U1C-VDD-Pad25) -> +3V3
- U1 pad 26: unconnected-(U1B-PF6-Pad26) -> /MCU2/QSPIMEM/QUADSPI_BK1_IO3
- U1 pad 27: unconnected-(U1B-PF7-Pad27) -> /MCU2/QSPIMEM/QUADSPI_BK1_IO2
- U1 pad 28: unconnected-(U1B-PF8-Pad28) -> /MCU2/QSPIMEM/QUADSPI_BK1_IO0
- U1 pad 29: unconnected-(U1B-PF9-Pad29) -> /MCU2/QSPIMEM/QUADSPI_BK1_IO1
- U1 pad 3: unconnected-(U1B-PE4-Pad3) -> /MCU2/100P_CONN/SAI1_FS
- U1 pad 30: unconnected-(U1B-PF10-Pad30) -> /MCU2/QSPIMEM/QUADSPI_BK1_CLK
- U1 pad 31: unconnected-(U1B-PH0-OSC_IN-Pad31) -> OSC_IN
- U1 pad 32: unconnected-(U1B-PH1-OSC_OUT-Pad32) -> OSC_OUT
- U1 pad 33: unconnected-(U1B-NRST-Pad33) -> H7NRST
- U1 pad 34: unconnected-(U1A-PC0-Pad34) -> /MCU2/100P_CONN/ADC_PC0
- U1 pad 35: unconnected-(U1A-PC1-Pad35) -> PC1
- U1 pad 38: unconnected-(U1C-VSSA-Pad38) -> GND
- U1 pad 39: unconnected-(U1C-VREF+-Pad39) -> Net-(U1C-VREF+)
- U1 pad 4: unconnected-(U1B-PE5-Pad4) -> /MCU2/100P_CONN/SAI1_SCK
- U1 pad 40: unconnected-(U1C-VDDA-Pad40) -> Net-(U1C-VDDA)
- U1 pad 41: unconnected-(U1A-PA0-Pad41) -> /MCU2/100P_CONN/ADC_PA0
- U1 pad 42: unconnected-(U1A-PA1-Pad42) -> PA1
- U1 pad 43: unconnected-(U1A-PA2-Pad43) -> PA2
- U1 pad 44: unconnected-(U1C-VDD-Pad44) -> +3V3
- U1 pad 45: unconnected-(U1C-VSS-Pad45) -> GND
- U1 pad 46: unconnected-(U1A-PA3-Pad46) -> /MCU2/100P_CONN/ADC_PA3
- U1 pad 47: unconnected-(U1C-VSS-Pad47) -> GND
- U1 pad 48: unconnected-(U1C-VDD-Pad48) -> +3V3
- U1 pad 49: unconnected-(U1A-PA4-Pad49) -> /MCU2/100P_CONN/DAC_ADC_PA4
- U1 pad 5: unconnected-(U1B-PE6-Pad5) -> /MCU2/100P_CONN/SAI1_SD
- U1 pad 50: unconnected-(U1A-PA5-Pad50) -> /MCU2/100P_CONN/DAC_ADC_PA5
- U1 pad 51: unconnected-(U1A-PA6-Pad51) -> /MCU2/100P_CONN/ADC_PA6
- U1 pad 52: unconnected-(U1A-PA7-Pad52) -> PA7
- U1 pad 53: unconnected-(U1A-PC4-Pad53) -> PC4
- U1 pad 54: unconnected-(U1A-PC5-Pad54) -> PC5
- U1 pad 55: unconnected-(U1A-PB0-Pad55) -> /MCU2/100P_CONN/ADC_PB0
- U1 pad 56: unconnected-(U1A-PB1-Pad56) -> /MCU2/100P_CONN/ADC_PB1
- U1 pad 57: unconnected-(U1A-PB2-Pad57) -> /MCU2/100P_CONN/GPIO_PB2
- U1 pad 58: unconnected-(U1B-PF11-Pad58) -> PF11
- U1 pad 59: unconnected-(U1B-PF12-Pad59) -> PF12
- U1 pad 6: unconnected-(U1C-VSS-Pad6) -> GND
- U1 pad 60: unconnected-(U1B-PF13-Pad60) -> PF13
- U1 pad 61: unconnected-(U1B-PF14-Pad61) -> PF14
- U1 pad 62: unconnected-(U1B-PF15-Pad62) -> PF15
- U1 pad 63: unconnected-(U1B-PG0-Pad63) -> /MCU2/100P_CONN/GPIO_PG0
- U1 pad 64: unconnected-(U1C-VSS-Pad64) -> GND
- U1 pad 65: unconnected-(U1C-VDD-Pad65) -> +3V3
- U1 pad 66: unconnected-(U1B-PG1-Pad66) -> /MCU2/100P_CONN/GPIO_PG1
- U1 pad 67: unconnected-(U1B-PE7-Pad67) -> /MCU2/100P_CONN/GPIO_PE7
- U1 pad 68: unconnected-(U1B-PE8-Pad68) -> /MCU2/100P_CONN/MOTOR_CH1N
- U1 pad 69: unconnected-(U1B-PE9-Pad69) -> /MCU2/100P_CONN/MOTOR_CH1
- U1 pad 7: unconnected-(U1C-VDD-Pad7) -> +3V3
- U1 pad 70: unconnected-(U1C-VSS-Pad70) -> GND
- U1 pad 71: unconnected-(U1C-VDD-Pad71) -> +3V3
- U1 pad 72: unconnected-(U1B-PE10-Pad72) -> /MCU2/100P_CONN/MOTOR_CH2N
- U1 pad 73: unconnected-(U1B-PE11-Pad73) -> /MCU2/100P_CONN/MOTOR_CH2
- U1 pad 74: unconnected-(U1B-PE12-Pad74) -> /MCU2/100P_CONN/MOTOR_CH3N
- U1 pad 75: unconnected-(U1B-PE13-Pad75) -> /MCU2/100P_CONN/MOTOR_CH3
- U1 pad 76: unconnected-(U1B-PE14-Pad76) -> /MCU2/100P_CONN/MOTOR_CH4
- U1 pad 77: unconnected-(U1B-PE15-Pad77) -> /MCU2/100P_CONN/MOTOR_BKIN
- U1 pad 78: unconnected-(U1A-PB10-Pad78) -> PB10
- U1 pad 79: unconnected-(U1A-PB11-Pad79) -> PB11
- U1 pad 8: unconnected-(U1C-VBAT-Pad8) -> +3V3
- U1 pad 80: unconnected-(U1C-VCAP-Pad80) -> Net-(C30-Pad1)
- U1 pad 81: unconnected-(U1C-VSS-Pad81) -> GND
- U1 pad 82: unconnected-(U1C-VDDLDO-Pad82) -> Net-(U1C-VFBSMPS)
- U1 pad 83: unconnected-(U1C-VSS-Pad83) -> GND
- U1 pad 84: unconnected-(U1C-VDD-Pad84) -> +3V3
- U1 pad 85: unconnected-(U1A-PB12-Pad85) -> SPI2_NSS
- U1 pad 86: unconnected-(U1A-PB13-Pad86) -> SPI2_SCK
- U1 pad 87: unconnected-(U1A-PB14-Pad87) -> SPI2_MISO
- U1 pad 88: unconnected-(U1A-PB15-Pad88) -> SPI2_MOSI
- U1 pad 89: unconnected-(U1A-PD8-Pad89) -> PD8
- U1 pad 90: unconnected-(U1A-PD9-Pad90) -> PD9
- U1 pad 91: unconnected-(U1A-PD10-Pad91) -> PD10
- U1 pad 92: unconnected-(U1C-VDD-Pad92) -> +3V3
- U1 pad 93: unconnected-(U1C-VSS-Pad93) -> GND
- U1 pad 94: unconnected-(U1A-PD11-Pad94) -> PD11
- U1 pad 95: unconnected-(U1A-PD12-Pad95) -> PD12
- U1 pad 96: unconnected-(U1A-PD13-Pad96) -> PD13
- U1 pad 97: unconnected-(U1A-PD14-Pad97) -> PD14
- U1 pad 98: unconnected-(U1A-PD15-Pad98) -> PD15
- U1 pad 99: unconnected-(U1C-VDD-Pad99) -> +3V3
Routing:
- net GND: track 0.00 -> 233.3 mm, vias 0 -> 139
- net 3V3PROGRAMMER: track 0.00 -> 220.1 mm, vias 0 -> 3
- net Net-(D1-A1): track 0.00 -> 153.4 mm, vias 0 -> 1
- net Net-(D1-A2): track 0.00 -> 144.2 mm, vias 0 -> 1
- net +3V3: track 0.00 -> 143.3 mm, vias 0 -> 51
- net Net-(U1C-VFBSMPS): track 0.00 -> 97.5 mm, vias 0 -> 4
- net Net-(D4-Pad2): track 0.00 -> 93.0 mm, vias 0 -> 1
- net 5VHSSoC: track 0.00 -> 79.6 mm, vias 0 -> 4
- net PA2: track 0.00 -> 71.5 mm, vias 0 -> 2
- net PA7: track 0.00 -> 66.1 mm, vias 0 -> 2
- net PC4: track 0.00 -> 65.4 mm, vias 0 -> 2
- net PC5: track 0.00 -> 64.7 mm, vias 0 -> 2
- net H7SWO: track 0.00 -> 63.7 mm, vias 0 -> 1
- net Net-(J6-Pad37): track 0.00 -> 56.4 mm, vias 0 -> 1
- net Net-(J6-Pad12): track 0.00 -> 55.6 mm, vias 0 -> 1
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- added copper zone on In2.Cu, net +3V3
- added copper zone on B.Cu, net GND
- added copper zone on F.Cu, net GND
- added copper zone on In1.Cu, net GND
Other:
- copper layers 2 -> 4
- board text added: "CLOSE IF TOTEM POLE TERMINATOR"
- board text added: "Check out our platform! https://github.com/MakeyDooey"
- board text added: "Designed by Dom Murphy https://github.com/DomMurphy-git"
- board text added: "G0_UART/SWD"
- board text added: "H7 PIN HEADER VS STM32G0 PINS"
- board text added: "MakeyDooey Main Totem V1"
- board text added: "USER LEDS"

Commit message: Rerouting layout to resolve collision issues
Parts:
- R46, R47, R48, R49, R50, R51, R52, R53, R55, R56, RN10, RN2, RN3, RN5, RN6, RN7, RN8, RN9: moved to B.Cu
- moved RN5 162.3 mm to (87.4, 105.4), turned to 180 degrees
- moved RN10 152.3 mm to (95.8, 105.1), turned to 180 degrees
- moved RN3 150.4 mm to (91.9, 105.4), turned to 180 degrees
- moved RN6 147.1 mm to (83.1, 105.3), turned to 180 degrees
- moved RN9 144.7 mm to (99.9, 105.0), turned to 180 degrees
- moved R52 144.5 mm to (85.4, 101.1), turned to -90 degrees
- moved RN2 136.6 mm to (103.8, 105.1), turned to 180 degrees
- moved R48 136.4 mm to (87.6, 101.2), turned to -90 degrees
- moved R49 133.3 mm to (89.8, 101.2), turned to -90 degrees
- moved R55 130.8 mm to (97.5, 102.1), turned to 180 degrees
- moved R51 129.0 mm to (92.0, 101.2), turned to -90 degrees
- moved R47 128.5 mm to (97.5, 100.0), turned to 180 degrees
- moved R50 128.1 mm to (94.3, 101.2), turned to -90 degrees
- moved R46 126.4 mm to (101.5, 100.0), turned to 180 degrees
- moved R56 126.2 mm to (101.4, 102.2), turned to 180 degrees
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- renumbered 3V3HPSoC to 3V3HPSoC1, 3V3HSSoC to 3V3HSSoC1, 3V3SoC to 3V3SoC1, GND to GND1, H7_UART/SWD to H7_UART/SWD1, UH_OH to UH_OH1, USER to USER1
Connections:
- J5 pad 10: Net-(J5-Pad10) -> unconnected-(J5-Pad10)
- J5 pad 12: Net-(J5-Pad12) -> unconnected-(J5-Pad12)
- J5 pad 13: Net-(J5-Pad13) -> unconnected-(J5-Pad13)
- J5 pad 14: Net-(J5-Pad14) -> unconnected-(J5-Pad14)
- J5 pad 15: USART6_CTS -> unconnected-(J5-Pad15)
- J5 pad 17: Net-(J5-Pad17) -> unconnected-(J5-Pad17)
- J5 pad 18: Net-(J5-Pad18) -> unconnected-(J5-Pad18)
- J5 pad 19: Net-(J5-Pad19) -> unconnected-(J5-Pad19)
- J5 pad 20: Net-(J5-Pad20) -> unconnected-(J5-Pad20)
- J5 pad 22: Net-(J5-Pad22) -> unconnected-(J5-Pad22)
- J5 pad 25: Net-(J5-Pad25) -> unconnected-(J5-Pad25)
- J5 pad 27: Net-(J5-Pad27) -> unconnected-(J5-Pad27)
- J5 pad 28: Net-(J5-Pad28) -> unconnected-(J5-Pad28)
- J5 pad 29: Net-(J5-Pad29) -> unconnected-(J5-Pad29)
- J5 pad 3: USB_D+ -> unconnected-(J5-Pad3)
- J5 pad 30: Net-(J5-Pad30) -> unconnected-(J5-Pad30)
- J5 pad 32: Net-(J5-Pad32) -> unconnected-(J5-Pad32)
- J5 pad 33: Net-(J5-Pad33) -> unconnected-(J5-Pad33)
- J5 pad 35: Net-(J5-Pad35) -> unconnected-(J5-Pad35)
- J5 pad 37: Net-(J5-Pad37) -> unconnected-(J5-Pad37)
- J5 pad 39: PD13 -> unconnected-(J5-Pad39)
- J5 pad 43: PD12 -> unconnected-(J5-Pad43)
- J5 pad 5: USB_D- -> unconnected-(J5-Pad5)
- J5 pad 65: Net-(J5-Pad65) -> unconnected-(J5-Pad65)
- J5 pad 67: Net-(J5-Pad67) -> unconnected-(J5-Pad67)
- J5 pad 69: Net-(J5-Pad69) -> unconnected-(J5-Pad69)
- J5 pad 7: Net-(J5-Pad7) -> unconnected-(J5-Pad7)
- J5 pad 75: Net-(J5-Pad75) -> unconnected-(J5-Pad75)
- J5 pad 77: Net-(J5-Pad77) -> unconnected-(J5-Pad77)
- J5 pad 78: /MCU2/100P_CONN/ADC_PA0 -> unconnected-(J5-Pad78)
- J5 pad 79: Net-(J5-Pad79) -> unconnected-(J5-Pad79)
- J5 pad 8: Net-(J5-Pad8) -> unconnected-(J5-Pad8)
- J5 pad 83: Net-(J5-Pad83) -> unconnected-(J5-Pad83)
- J5 pad 85: Net-(J5-Pad85) -> unconnected-(J5-Pad85)
- J5 pad 9: USART6_RX -> unconnected-(J5-Pad9)
- R46 pad 1: /MCU2/100P_CONN/GPIO_PA8_CLKOUT -> unconnected-(R46-Pad1)
- R46 pad 2: Net-(J5-Pad7) -> unconnected-(R46-Pad2)
- R47 pad 1: USART6_TX -> unconnected-(R47-Pad1)
- R47 pad 2: Net-(J5-Pad13) -> unconnected-(R47-Pad2)
- R48 pad 2: USART6_RX -> unconnected-(R48-Pad2)
- R49 pad 2: USART6_CTS -> unconnected-(R49-Pad2)
- R50 pad 2: PD13 -> unconnected-(R50-Pad2)
- R51 pad 2: PD12 -> unconnected-(R51-Pad2)
- R52 pad 2: /MCU2/100P_CONN/MOTOR_BKIN -> unconnected-(R52-Pad2)
- R55 pad 1: /MCU2/100P_CONN/GPIO_PF1 -> unconnected-(R55-Pad1)
- R55 pad 2: Net-(J5-Pad20) -> unconnected-(R55-Pad2)
- R56 pad 1: /MCU2/100P_CONN/GPIO_PF0 -> unconnected-(R56-Pad1)
- R56 pad 2: Net-(J5-Pad18) -> unconnected-(R56-Pad2)
- RN10 pad 1: Net-(J5-Pad14) -> unconnected-(RN10-Pad1)
- RN10 pad 2: Net-(J5-Pad12) -> unconnected-(RN10-Pad2)
- RN10 pad 3: Net-(J5-Pad10) -> unconnected-(RN10-Pad3)
- RN10 pad 4: Net-(J5-Pad8) -> unconnected-(RN10-Pad4)
- RN10 pad 5: /MCU2/100P_CONN/SAI1_MCLK -> unconnected-(RN10-Pad5)
- RN10 pad 6: /MCU2/100P_CONN/SAI1_FS -> unconnected-(RN10-Pad6)
- RN10 pad 7: /MCU2/100P_CONN/SAI1_SCK -> unconnected-(RN10-Pad7)
- RN10 pad 8: /MCU2/100P_CONN/SAI1_SD -> unconnected-(RN10-Pad8)
- RN2 pad 1: Net-(J5-Pad37) -> unconnected-(RN2-Pad1)
- RN2 pad 2: Net-(J5-Pad35) -> unconnected-(RN2-Pad2)
- RN2 pad 3: Net-(J5-Pad33) -> unconnected-(RN2-Pad3)
- RN2 pad 4: Net-(J5-Pad29) -> unconnected-(RN2-Pad4)
- RN2 pad 5: /MCU2/100P_CONN/GPIO_PG3 -> unconnected-(RN2-Pad5)
- RN2 pad 6: /MCU2/100P_CONN/GPIO_PG2 -> unconnected-(RN2-Pad6)
- RN2 pad 7: PD15 -> unconnected-(RN2-Pad7)
- RN2 pad 8: PD14 -> unconnected-(RN2-Pad8)
- RN3 pad 1: Net-(J5-Pad27) -> unconnected-(RN3-Pad1)
- RN3 pad 2: Net-(J5-Pad25) -> unconnected-(RN3-Pad2)
- RN3 pad 3: Net-(J5-Pad19) -> unconnected-(RN3-Pad3)
- RN3 pad 4: Net-(J5-Pad17) -> unconnected-(RN3-Pad4)
- RN3 pad 5: USART6_RTS -> unconnected-(RN3-Pad5)
- RN3 pad 6: /MCU2/100P_CONN/GPIO_PG6 -> unconnected-(RN3-Pad6)
- RN3 pad 7: /MCU2/100P_CONN/GPIO_PG5 -> unconnected-(RN3-Pad7)
- RN3 pad 8: /MCU2/100P_CONN/GPIO_PG4 -> unconnected-(RN3-Pad8)
- RN5 pad 1: /MCU2/100P_CONN/MOTOR_BKIN -> unconnected-(RN5-Pad1)
- RN5 pad 2: /MCU2/100P_CONN/MOTOR_CH4 -> unconnected-(RN5-Pad2)
- RN5 pad 3: /MCU2/100P_CONN/MOTOR_CH3 -> unconnected-(RN5-Pad3)
- RN5 pad 4: /MCU2/100P_CONN/MOTOR_CH3N -> unconnected-(RN5-Pad4)
- RN5 pad 5: Net-(J5-Pad75) -> unconnected-(RN5-Pad5)
- RN5 pad 6: Net-(J5-Pad69) -> unconnected-(RN5-Pad6)
- RN5 pad 7: Net-(J5-Pad67) -> unconnected-(RN5-Pad7)
- RN5 pad 8: Net-(J5-Pad65) -> unconnected-(RN5-Pad8)
- RN6 pad 1: /MCU2/100P_CONN/MOTOR_CH2 -> unconnected-(RN6-Pad1)
- RN6 pad 2: /MCU2/100P_CONN/MOTOR_CH2N -> unconnected-(RN6-Pad2)
- RN6 pad 3: /MCU2/100P_CONN/MOTOR_CH1 -> unconnected-(RN6-Pad3)
- RN6 pad 4: /MCU2/100P_CONN/MOTOR_CH1N -> unconnected-(RN6-Pad4)
- RN6 pad 5: Net-(J5-Pad85) -> unconnected-(RN6-Pad5)
- RN6 pad 6: Net-(J5-Pad83) -> unconnected-(RN6-Pad6)
- RN6 pad 7: Net-(J5-Pad79) -> unconnected-(RN6-Pad7)
- RN6 pad 8: Net-(J5-Pad77) -> unconnected-(RN6-Pad8)
- RN7 pad 1: /MCU2/100P_CONN/GPIO_PE7 -> Net-(J5-Pad87)
- RN7 pad 2: /MCU2/100P_CONN/GPIO_PG1 -> Net-(J5-Pad89)
- RN7 pad 3: /MCU2/100P_CONN/GPIO_PG0 -> Net-(J5-Pad93)
- RN7 pad 4: PF15 -> Net-(J5-Pad95)
- RN7 pad 5: Net-(J5-Pad95) -> PF15
- RN7 pad 6: Net-(J5-Pad93) -> /MCU2/100P_CONN/GPIO_PG0
- RN7 pad 7: Net-(J5-Pad89) -> /MCU2/100P_CONN/GPIO_PG1
- RN7 pad 8: Net-(J5-Pad87) -> /MCU2/100P_CONN/GPIO_PE7
- RN8 pad 1: PF14 -> Net-(J5-Pad97)
- RN8 pad 2: PF13 -> Net-(J5-Pad99)
- RN8 pad 3: PF12 -> Net-(J5-Pad96)
- RN8 pad 4: PF11 -> Net-(J5-Pad94)
- RN8 pad 5: Net-(J5-Pad94) -> PF11
- RN8 pad 6: Net-(J5-Pad96) -> PF12
- RN8 pad 7: Net-(J5-Pad99) -> PF13
- RN8 pad 8: Net-(J5-Pad97) -> PF14
- RN9 pad 1: Net-(J5-Pad32) -> unconnected-(RN9-Pad1)
- RN9 pad 2: Net-(J5-Pad30) -> unconnected-(RN9-Pad2)
- RN9 pad 3: Net-(J5-Pad28) -> unconnected-(RN9-Pad3)
- RN9 pad 4: Net-(J5-Pad22) -> unconnected-(RN9-Pad4)
- RN9 pad 5: /MCU2/100P_CONN/GPIO_PF2 -> unconnected-(RN9-Pad5)
- RN9 pad 6: /MCU2/100P_CONN/GPIO_PF3 -> unconnected-(RN9-Pad6)
- RN9 pad 7: /MCU2/100P_CONN/GPIO_PF4 -> unconnected-(RN9-Pad7)
- RN9 pad 8: /MCU2/100P_CONN/GPIO_PF5 -> unconnected-(RN9-Pad8)
Routing:
- net 5VHPSoC: track 17.3 -> 67.4 mm, vias 0 -> 2
- net Net-(J5-Pad45): track 0.00 -> 48.2 mm
- net Net-(J5-Pad47): track 0.00 -> 46.1 mm
- net Net-(J5-Pad49): track 0.00 -> 44.3 mm
- net GND: track 233.3 -> 276.5 mm, vias 139 -> 157
- net +3V3: track 143.3 -> 186.3 mm, vias 51 -> 72
- net Net-(J5-Pad53): track 0.00 -> 41.7 mm
- net Net-(J5-Pad55): track 0.00 -> 34.1 mm, vias 0 -> 2
- net /MCU2/100P_CONN/ADC_PC0: track 0.00 -> 32.8 mm, vias 0 -> 2
- net Net-(J5-Pad57): track 0.00 -> 31.9 mm
- net Net-(J5-Pad59): track 0.00 -> 30.6 mm, vias 0 -> 2
- net Net-(J5-Pad87): track 0.00 -> 28.4 mm, vias 0 -> 1
- net Net-(J5-Pad63): track 0.00 -> 27.3 mm, vias 0 -> 2
- net Net-(J5-Pad97): track 0.00 -> 26.2 mm, vias 0 -> 1
- net Net-(J5-Pad89): track 0.00 -> 25.6 mm, vias 0 -> 1
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Other:
- board outline added: 143.9 x 76.1 mm
- board text added: "Components Pending V2"

Commit message: Adding Gerber and CAD files
Parts:
- renumbered 3V3HPSoC1 to 3V3HPSoC, 3V3HSSoC1 to 3V3HSSoC, 3V3SoC1 to 3V3SoC, GND1 to GND, H7RST1 to H7RST, PROG1 to PROG, UH_OH1 to UH_OH, USER1 to USER
Routing:
- net GND: vias 157 -> 200

Commit message: Computer Vision Module Alterations
Parts:
- moved G*** 1.10 mm to (107.9, 59.4)
- renumbered H7RST to H7RST1, H7_UART/SWD1 to H7_UART/SWD
Connections:
- C72 pad 1: 3V3PROGRAMMER -> 3V3MODULES
- C73 pad 1: 3V3PROGRAMMER -> 3V3MODULES
- C74 pad 1: 3V3MODULES -> 3V3PROGRAMMER
- C75 pad 1: 3V3MODULES -> 3V3PROGRAMMER
- R19 pad 1: 3V3PROGRAMMER -> 3V3MODULES
- R21 pad 1: 3V3PROGRAMMER -> 3V3MODULES
- U11 pad 3: 3V3PROGRAMMER -> 3V3MODULES
- U11 pad 5: 3V3PROGRAMMER -> 3V3MODULES
- U11 pad 6: 3V3MODULES -> 3V3PROGRAMMER
Routing:
- net 3V3MODULES: track 18.9 -> 51.9 mm
- net GND: track 276.5 -> 280.3 mm, vias 200 -> 202
- net 3V3PROGRAMMER: track 220.1 -> 217.3 mm
Other:
- board text added: "H7NRST"
