File: Schematics/ShamanLink_Rev1/maintotemheader.kicad_sch (KiCad schematic)
At the start: 9 parts, among them J5 Conn_ARM_SWD_TagConnect_TC203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

Commit message: Computer Vision Module Alterations
Other:
- note added: "This 3V3 CANNOT be the TagConnect connection. It is too high resistance to handle any power supply, you can use the Tagconnect for the signals, but you will need a jumper for the power and gnd connections."
Changed lines of the file:
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@@
 	(generator_version "9.0")
 	(paper "A4")
+	(text "This 3V3 CANNOT be the TagConnect connection. \nIt is too high resistance to handle any power supply, you can use the \nTagconnect for the signals, but you will need a jumper for the \npower and gnd connections. "
+		(exclude_from_sim no)
+		(at 178.562 70.612 0)
+		(effects
+			(font
+				(size 1.27 1.27)
+			)
+		)
+	)
 	(text "No need to implement these pull up and pull down\nresistors on the target board since they are already implemented \nhere. "
 		(exclude_from_sim no)
