File: Schematics/ShamanLink_Rev1/power.kicad_sch (KiCad schematic)
At the start: 17 parts, among them SW1 SW_Push, U3 AP7361C-33Y5-13, U4 PTPS2117DRLR

Commit message: Computer Vision Module Alterations
Other:
- note added: "In this configuration, you have the 3V3 as the priority supply."
Changed lines of the file:
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@@
+		)
+	)
+	(text "In this configuration, you have the 3V3 as the priority supply."
+		(exclude_from_sim no)
+		(at 229.108 130.81 0)
+		(effects
+			(font
+				(size 1.27 1.27)
+			)
 		)
 	)
