File: Schematics/TouchScreenModule_Rev1/TouchScreenModule_Rev1/power.kicad_sch (KiCad schematic)
At the start: 12 parts, among them J3 Screw_Terminal_01x02, U1 TPS562208DDCR

Commit message: CAD files and Schematic PDFs
Other:
- note added: "A 51kohm R used here irl"
- note added: "For these caps you didnt have 22uF 0805 caps, so you stacked two 10uF caps on top each other."
Changed lines of the file:
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@@
 	(generator_version "9.0")
 	(paper "A4")
+	(text "For these caps you didnt have 22uF 0805 caps,\nso you stacked two 10uF caps on top each other. "
+		(exclude_from_sim no)
+		(at 93.726 83.566 0)
+		(effects
+			(font
+				(size 1.27 1.27)
+			)
+		)
+	)
+	(text "A 51kohm R used here irl"
+		(exclude_from_sim no)
+		(at 118.618 92.964 0)
+		(effects
+			(font
+				(size 1.27 1.27)
+			)
+		)
+	)
 	(junction
 		(at 135.89 86.36)
